File: pcb_files/Mbus.brd (EAGLE design)
At the start: 98.7 x 71.1 mm, 50 parts, among them IC1 NCP1117ST50T3G, IC3 ATMEGA2560-16AU, IC4 RTC_PCF8523T, J1 F-1X18-SIP-100-32Y, J2 USB_A_SMT_FEMALE, J3 USB_A_SMT_FEMALE, J4 USB_A_SMT_FEMALE, M1 SERVO, Q2 32.768, Y1 CSTCE16M0V53-R0 16MHZ

Commit message: Add resisters for 5V microcontroller to 3.3V pi pin header
Signed-off-by: AlonsoChate <alonsochate@sjtu.edu.cn>
Parts:
- added R2: 3.3k, SmartPrj:R0603-ROUND
- added R3: 1.6k, SmartPrj:R0603-ROUND
Connections:
- net GND: now also R2.1
- net TXD2: now also R2.2, R3.1, R3.2
Changed lines of the file:
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@@
 <drawing>
 <settings>
-<setting alwaysvectorfont="no"/>
+<setting alwaysvectorfont="yes"/>
 <setting verticaltext="up"/>
 </settings>
@@
 <attribute name="VALUE" x="-52.578" y="-8.636" size="0.6096" layer="27" font="vector" ratio="20" align="top-left"/>
 </element>
+<element name="R2" library="SmartPrj" package="R0603-ROUND" value="3.3k" x="-52.07" y="-12.954" smashed="yes">
+<attribute name="NAME" x="-52.959" y="-12.065" size="1.27" layer="25"/>
+<attribute name="VALUE" x="-52.959" y="-14.986" size="1.27" layer="27"/>
+</element>
+<element name="R3" library="SmartPrj" package="R0603-ROUND" value="1.6k" x="-52.07" y="-18.288" smashed="yes">
+<attribute name="NAME" x="-52.959" y="-17.399" size="1.27" layer="25"/>
+<attribute name="VALUE" x="-52.959" y="-20.32" size="1.27" layer="27"/>
+</element>
 </elements>
 <signals>
@@
 <contactref element="J3" pad="GND"/>
 <contactref element="J4" pad="GND"/>
+<contactref element="R2" pad="1"/>
 <wire x1="89.408" y1="19.558" x2="95.25" y2="33.02" width="0" layer="19" extent="1-1"/>
 <wire x1="88.072" y1="13.716" x2="89.408" y2="19.558" width="0" layer="19" extent="1-1"/>
@@
 <wire x1="-22.506" y1="-5.278" x2="-5.996" y2="-5.278" width="0" layer="19" extent="1-1"/>
 <wire x1="-39.016" y1="-5.278" x2="-22.506" y2="-5.278" width="0" layer="19" extent="1-1"/>
+<wire x1="-52.959" y1="-12.954" x2="-39.016" y2="-5.278" width="0" layer="19" extent="1-1"/>
 <wire x1="57.916" y1="66.808" x2="49.15" y2="45.918" width="0" layer="19" extent="1-1"/>
 </signal>
@@
 <via x="29.337" y="33.7566" extent="1-16" drill="0.35"/>
 <via x="26.8986" y="31.3182" extent="1-16" drill="0.35"/>
+<contactref element="R3" pad="2"/>
+<contactref element="R2" pad="2"/>
+<contactref element="R3" pad="1"/>
+<wire x1="-52.959" y1="-18.288" x2="-51.181" y2="-18.288" width="0" layer="19" extent="1-1"/>
+<wire x1="-51.181" y1="-12.954" x2="-51.181" y2="-18.288" width="0" layer="19" extent="1-1"/>
+<wire x1="4.318" y1="16.002" x2="-51.181" y2="-12.954" width="0" layer="19" extent="1-1"/>
 </signal>
 <signal name="PC0">
