File: pcb_files/Mbus.brd (EAGLE design)
At the start: 98.7 x 71.1 mm, 51 parts, among them IC1 NCP1117ST50T3G, IC3 ATMEGA2560-16AU, IC4 RTC_PCF8523T, J1 F-1X18-SIP-100-32Y, J2 USB_A_SMT_FEMALE, M1 SERVO, Q2 32.768, Y1 CSTCE16M0V53-R0 16MHZ

Commit message: gpio re-organize
Parts:
- removed C10: 10uF, microbuilder:0805-NO
- moved J3 132.6 mm to (74.2, 2.79), turned to 90 degrees
- moved R3 119.4 mm to (59.4, 24.4)
- moved R2 114.3 mm to (59.2, 13.5)
- moved FID4 93.6 mm to (1.78, 67.1)
- moved FID3 89.2 mm to (6.60, 66.5)
- moved J2 72.7 mm to (59.4, 1.27), turned to 90 degrees
- moved TESTPIN 72.1 mm to (91.4, 23.1), turned to 90 degrees
- moved R8 37.2 mm to (22.1, 25.4)
- moved POWER 33.8 mm to (20.8, 2.54)
- moved RESET 25.7 mm to (66.3, 19.8), turned to 270 degrees
- moved IC1 23.9 mm to (31.5, 11.2), turned to 0 degrees
- moved RN2 23.7 mm to (61.0, 61.7)
- moved J1 17.8 mm to (96.3, 47.0)
- moved C4 17.8 mm to (48.3, 29.2)
- moved SJ4 15.3 mm to (30.5, 28.7), flipped to the top
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Connections:
- new net GND3: IC3.81
- new net PD5: IC3.48, TESTPIN.6
- new net PD6: IC3.49, TESTPIN.7
- new net PD7: IC3.50, TESTPIN.8
- new net PJ2: IC3.65, J1.5
- new net RXD3: IC3.63, J1.7
- new net TXD3: IC3.64, J1.6
- new net VCC3: IC3.80
- net +5V: no longer C10.1, IC3.80
- net GND: no longer C10.2, IC3.81
- net PB3: no longer TESTPIN.5
- net PB4: no longer TESTPIN.6
- net PB5: no longer TESTPIN.7
- net PB6: no longer TESTPIN.8
- net PD4: now also TESTPIN.5; no longer J1.5
- net RXD0: now also PIHEADER.8; no longer TESTPIN.4
- net RXD1: now also TESTPIN.4; no longer J1.7
- net RXD2: no longer PIHEADER.8
- net SCL: now also TESTPIN.1; no longer TESTPIN.2
- net SDA: now also TESTPIN.2; no longer TESTPIN.1
- net TXD0: now also R3.1; no longer TESTPIN.3
- net TXD1: now also TESTPIN.3; no longer J1.6
- net TXD2: no longer R3.1
Routing:
- net RESET: track 133.0 -> 0.00 mm, vias 3 -> 0
- net GND: track 108.0 -> 0.00 mm, vias 3 -> 0
- net SCL: track 102.2 -> 0.00 mm, vias 1 -> 0
- net SDA: track 92.7 -> 0.00 mm, vias 4 -> 0
- net PB1: track 80.4 -> 0.00 mm
- net RXD2: track 77.0 -> 0.00 mm, vias 2 -> 0
- net TXD2: track 76.8 -> 0.00 mm, vias 2 -> 0
- net PB6: track 66.9 -> 0.00 mm, vias 2 -> 0
- net PB5: track 63.5 -> 0.00 mm, vias 2 -> 0
- net PB3: track 60.3 -> 0.00 mm, vias 2 -> 0
- net N$22: track 58.7 -> 0.00 mm, vias 1 -> 0
- net PB4: track 57.5 -> 0.00 mm, vias 2 -> 0
- net PISCL: track 55.5 -> 0.00 mm, vias 1 -> 0
- net PISDA: track 52.9 -> 0.00 mm, vias 1 -> 0
- net PD4: track 46.1 -> 0.00 mm
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
Commit message: route update
Parts:
- moved ICSP 21.3 mm to (19.6, 4.32)
- moved POWER 19.3 mm to (40.1, 3.56)
- moved SJ3 11.5 mm to (30.0, 32.3), flipped to the bottom
- moved SJ4 8.98 mm to (38.6, 32.5), flipped to the bottom
- moved L 8.59 mm to (44.7, 23.4)
- moved PC2 8.33 mm to (35.3, 22.6)
- moved D3 6.14 mm to (49.8, 17.8), flipped to the bottom, turned to 180 degrees
- moved FD1 4.75 mm to (68.8, 54.6)
- moved ON 4.38 mm to (49.0, 22.1)
- moved R7 4.07 mm to (46.7, 44.5)
- moved C9 2.87 mm to (46.0, 39.9)
- moved D1 2.55 mm to (72.4, 11.9)
- moved TESTPIN 2.17 mm to (90.7, 21.1)
- moved R8 2.09 mm to (21.6, 23.4)
- moved R3 1.93 mm to (58.7, 26.2)
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Connections:
- removed net PJ2: IC3.65, J1.5
- net PD7: now also J1.5
- net RXD3: no longer IC3.63
- net TXD3: no longer IC3.64
Routing:
- net +5V: track 0.00 -> 213.3 mm, vias 0 -> 19
- net GND: track 0.00 -> 133.4 mm, vias 0 -> 6
- net RESET: track 0.00 -> 114.0 mm, vias 0 -> 2
- net TXD2: track 0.00 -> 80.2 mm, vias 0 -> 3
- net PB2: track 0.00 -> 67.1 mm
- net PB1: track 0.00 -> 61.6 mm, vias 0 -> 2
- net TXD1: track 0.00 -> 61.2 mm
- net RXD0: track 0.00 -> 61.0 mm, vias 0 -> 1
- net SCL: track 0.00 -> 60.1 mm
- net PB3: track 0.00 -> 60.0 mm, vias 0 -> 2
- net VIN: track 0.00 -> 55.7 mm
- net SDA: track 0.00 -> 53.5 mm
- net PISDA: track 0.00 -> 52.3 mm, vias 0 -> 1
- net PISCL: track 0.00 -> 49.1 mm, vias 0 -> 1
- net PC5: track 0.00 -> 40.8 mm
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