File: pcb_files/Mbus_1.3.brd (EAGLE design)
At the start: 101.6 x 71.1 mm, 49 parts, among them IC1 NCP1117ST50T3G, IC3 ATMEGA2560-16AU, IC4 RTC_PCF8523T, J1 F-1X18-SIP-100-32Y, J2 USB_A_SMT_FEMALE, M1 SERVO, Q1 BSS138, Q2 32.768, Q3 BSS138, Y1 CSTCE16M0V53-R0 16MHZ

Commit message: Trial on polygon
Signed-off-by: Yiteng Cai <alonsochate@umich.edu>
Parts:
- moved R3 7.09 mm to (52.1, 30.0), turned to 270 degrees
- moved Q1 3.96 mm to (54.2, 26.7), turned to 270 degrees
- moved R14 3.17 mm to (56.3, 34.3)
- moved Q3 2.96 mm to (51.9, 36.2), turned to 0 degrees
- moved R7 1.96 mm to (36.5, 33.1), turned to 180 degrees
- moved C9 0.28 mm to (34.5, 30.2)
Routing:
- net PL3: track 51.2 -> 0.00 mm, vias 6 -> 0
- net +3V3: track 103.6 -> 57.3 mm
- net RXD3: track 41.6 -> 0.00 mm, vias 2 -> 0
- net VIN: track 48.2 -> 27.0 mm
- net RXD0: track 72.9 -> 93.4 mm
- net PWRIN: track 12.0 -> 0.00 mm
- net GND: track 66.8 -> 60.9 mm, vias 11 -> 8
- net PD4: track 49.0 -> 43.4 mm
- net RESET: track 113.3 -> 110.2 mm
- net TXD3: track 45.5 -> 42.9 mm
- net PD7: track 129.3 -> 131.5 mm
- net TXD0: track 76.1 -> 77.1 mm
- net 5V: track 2.59 -> 3.38 mm
- net SCL: track 96.6 -> 96.3 mm, vias 3 -> 2
- added copper zone on layer 1, net +3V3
- added copper zone on layer 1, net VIN

Commit message: Modify the npn transistor and board layout for 1.2
Signed-off-by: Yiteng Cai <alonsochate@umich.edu>
Parts:
- removed M1: SERVO, SparkFun-Electromechanical:1X03
- moved R2 9.25 mm to (54.7, 31.6), turned to 0 degrees
- moved R3 4.48 mm to (48.5, 27.2), turned to 90 degrees
- moved R7 2.57 mm to (38.9, 33.9)
- moved Q1 2.43 mm to (52.3, 28.2)
- moved R15 1.69 mm to (50.2, 31.6), turned to 180 degrees
- moved R14 0.94 mm to (57.0, 35.0)
- moved C9 0.93 mm to (34.8, 31.1)
Connections:
- net +5V: no longer M1.2
- net GND: no longer M1.3
- net PL3: no longer M1.1
Routing:
- net RXD0: track 93.4 -> 78.1 mm, vias 1 -> 2
- net PD7: track 131.5 -> 140.4 mm, vias 2 -> 1
- net TXD0: track 77.1 -> 83.8 mm
- net +5V: track 0.00 -> 3.49 mm, vias 0 -> 2
- net N$10: track 6.24 -> 8.25 mm
- net +3V3: track 57.3 -> 58.2 mm
