File: pcb_files/Mbus_1.2.sch (EAGLE design)
At the start: 50 parts, among them IC1 NCP1117ST50T3G, IC3 ATMEGA2560-16AU, IC4 RTC_PCF8523T, J1 F-1X18-SIP-100-32Y, J2 USB_A_SMT_FEMALE, Q1 BSS138, Q2 32.768, Q3 BSS138, T1 2N3904, Y1 CSTCE16M0V53-R0 16MHZ

Commit message: Save
Signed-off-by: Yiteng Cai <alonsochate@umich.edu>
Connections:
- new net N$12: PIHEADER.RXI/GP15, Q3.S, R15.1
- new net N$5: PIHEADER.TXO/GP14, Q1.S, R3.1
- net RXD0: no longer PIHEADER.RXI/GP15, Q3.S, R15.1
- net TXD0: no longer PIHEADER.TXO/GP14, Q1.S, R3.1
Changed lines of the file:
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@@
 </variantdefs>
 <classes>
-<class number="0" name="default" width="0.2032" drill="0.4064">
-<clearance class="0" value="0.2032"/>
+<class number="0" name="default" width="0.2032" drill="0.3048">
+<clearance class="0" value="0.254"/>
 </class>
-<class number="1" name="power" width="0.8128" drill="0.8128">
+<class number="1" name="power" width="0.8128" drill="0.8636">
 <clearance class="1" value="0.254"/>
 </class>
-<class number="2" name="gnd" width="0.6096" drill="0.6096">
+<class number="2" name="gnd" width="0.6096" drill="0.6604">
 <clearance class="2" value="0.254"/>
 </class>
-<class number="3" name="power usb" width="0.8128" drill="0.8128">
+<class number="3" name="power usb" width="0.8128" drill="0.8636">
 <clearance class="3" value="0.254"/>
 </class>
@@
 </segment>
 <segment>
-<pinref part="Q1" gate="G$1" pin="S"/>
-<wire x1="340.36" y1="93.98" x2="332.74" y2="93.98" width="0.1524" layer="91"/>
-<pinref part="R3" gate="G$1" pin="1"/>
-<wire x1="332.74" y1="93.98" x2="302.26" y2="93.98" width="0.1524" layer="91"/>
-<wire x1="332.74" y1="96.52" x2="332.74" y2="93.98" width="0.1524" layer="91"/>
-<junction x="332.74" y="93.98"/>
-<pinref part="PIHEADER" gate="G$1" pin="TXO/GP14"/>
-</segment>
-<segment>
 <wire x1="350.52" y1="66.04" x2="360.68" y2="66.04" width="0.1524" layer="91"/>
 <wire x1="360.68" y1="66.04" x2="370.84" y2="66.04" width="0.1524" layer="91"/>
@@
 </segment>
 <segment>
-<wire x1="322.58" y1="91.44" x2="322.58" y2="66.04" width="0.1524" layer="91"/>
-<wire x1="322.58" y1="66.04" x2="332.74" y2="66.04" width="0.1524" layer="91"/>
-<pinref part="Q3" gate="G$1" pin="S"/>
-<pinref part="R15" gate="G$1" pin="1"/>
-<wire x1="332.74" y1="66.04" x2="340.36" y2="66.04" width="0.1524" layer="91"/>
-<wire x1="332.74" y1="68.58" x2="332.74" y2="66.04" width="0.1524" layer="91"/>
-<junction x="332.74" y="66.04"/>
-<pinref part="PIHEADER" gate="G$1" pin="RXI/GP15"/>
-<wire x1="302.26" y1="91.44" x2="322.58" y2="91.44" width="0.1524" layer="91"/>
-</segment>
-<segment>
 <pinref part="Q1" gate="G$1" pin="D"/>
 <pinref part="R2" gate="G$1" pin="1"/>
@@
 </segment>
 </net>
+<net name="N$5" class="0">
+<segment>
+<pinref part="Q1" gate="G$1" pin="S"/>
+<pinref part="PIHEADER" gate="G$1" pin="TXO/GP14"/>
+<wire x1="340.36" y1="93.98" x2="332.74" y2="93.98" width="0.1524" layer="91"/>
+<pinref part="R3" gate="G$1" pin="1"/>
+<wire x1="332.74" y1="93.98" x2="302.26" y2="93.98" width="0.1524" layer="91"/>
+<wire x1="332.74" y1="96.52" x2="332.74" y2="93.98" width="0.1524" layer="91"/>
+<junction x="332.74" y="93.98"/>
+</segment>
+</net>
+<net name="N$12" class="0">
+<segment>
+<pinref part="Q3" gate="G$1" pin="S"/>
+<wire x1="340.36" y1="66.04" x2="332.74" y2="66.04" width="0.1524" layer="91"/>
+<wire x1="332.74" y1="66.04" x2="322.58" y2="66.04" width="0.1524" layer="91"/>
+<wire x1="322.58" y1="66.04" x2="322.58" y2="91.44" width="0.1524" layer="91"/>
+<pinref part="PIHEADER" gate="G$1" pin="RXI/GP15"/>
+<wire x1="322.58" y1="91.44" x2="302.26" y2="91.44" width="0.1524" layer="91"/>
+<pinref part="R15" gate="G$1" pin="1"/>
+<wire x1="332.74" y1="68.58" x2="332.74" y2="66.04" width="0.1524" layer="91"/>
+<junction x="332.74" y="66.04"/>
+</segment>
+</net>

Commit message: Create gerber files
Signed-off-by: Yiteng Cai <alonsochate@umich.edu>
Connections:
- removed net RXD2: IC3.PH0(RXD2)
- removed net TXD2: IC3.PH1(TXD2)
Changed lines of the file:
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@@
-</segment>
-</net>
-<net name="RXD2" class="0">
-<segment>
-<wire x1="91.44" y1="-12.7" x2="104.14" y2="-12.7" width="0.1524" layer="91"/>
-<label x="93.98" y="-12.065" size="1.778" layer="95"/>
-<pinref part="IC3" gate="1" pin="PH0(RXD2)"/>
-</segment>
-</net>
-<net name="TXD2" class="0">
-<segment>
-<wire x1="91.44" y1="-10.16" x2="104.14" y2="-10.16" width="0.1524" layer="91"/>
-<label x="93.98" y="-9.525" size="1.778" layer="95"/>
-<pinref part="IC3" gate="1" pin="PH1(TXD2)"/>
 </segment>
 </net>
