File: pcb_files/Mbus_1.3.sch (EAGLE design)
At the start: 50 parts, among them IC1 NCP1117ST50T3G, IC3 ATMEGA2560-16AU, IC4 RTC_PCF8523T, J1 F-1X18-SIP-100-32Y, J2 USB_A_SMT_FEMALE, Q1 BSS138, Q2 32.768, Q3 BSS138, T1 2N3904, Y1 CSTCE16M0V53-R0 16MHZ

Commit message: 328
Parts:
- removed R17: 1k, SmartPrj:R-EU_R0603
- removed T1: 2N3904, transistor:2N3904
- added M1: SERVO, SparkFun-Electromechanical:SERVO
Connections:
- removed net N$1: IC3.PK7(ADC15/PCINT23), R16.1
- removed net N$12: PIHEADER.RXI/GP15, Q3.S, R15.1
- removed net N$4: R16.2, T1.B
- removed net N$5: PIHEADER.TXO/GP14, Q1.S, R3.1
- removed net OUT: PIHEADER.SCL/GP3\, R17.1, T1.C
- new net RXD2: IC3.PH0(RXD2)
- new net TXD2: IC3.PH1(TXD2)
- net +3V3: now also R16.2
- net +5V: now also M1.V+; no longer R17.2
- net GND: now also M1.GND; no longer T1.E
- net PD7: now also PIHEADER.SCL/GP3\, R16.1
- net PL3: now also M1.SIG
- net RXD0: now also PIHEADER.RXI/GP15, Q3.S, R15.1
- net TXD0: now also PIHEADER.TXO/GP14, Q1.S, R3.1
Other:
- moved on the sheet: R16
