File: pcb_files/Mbus_3.0.brd (EAGLE design)
At the start: 113 x 78.7 mm, 39 parts, among them IC1 NCP1117ST50T3G, J1 F-1X18-SIP-100-32Y, J2 USB_A_SMT_FEMALE, Q1 BSS138, Q3 BSS138, Q4 CSM-7X-DU, T1 2N3904, U1 ATMEGA328P-AU, X1 POWERSUPPLY_DC21MMX

Commit message: delete some traces
Signed-off-by: Yiteng Cai <alonsochate@umich.edu>
Routing:
- net +5V: track 42.9 -> 34.8 mm
Other:
- board text added: "MBUS BOARD v3.0"
- board text removed: "MBUS BOARD v2.0"
Changed lines of the file:
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@@
 <drawing>
 <settings>
-<setting alwaysvectorfont="no"/>
+<setting alwaysvectorfont="yes"/>
 <setting verticaltext="up"/>
 </settings>
@@
 <hole x="66.802" y="4.064" drill="5.08"/>
 <text x="90.03791875" y="1.272540625" size="1.778" layer="25">MBUS BOARD
-      v2.0</text>
+      v3.0</text>
 </plain>
 <attributes>
@@
 <contactref element="C1" pad="1"/>
 <contactref element="R6" pad="2"/>
-<wire x1="70.8152" y1="48.4632" x2="74.9808" y2="48.4632" width="0.2032" layer="1"/>
-<wire x1="70.7136" y1="48.3616" x2="70.8152" y2="48.4632" width="0.2032" layer="1"/>
-<wire x1="74.9808" y1="48.4632" x2="75.0468" y2="48.46828125" width="0.2032" layer="1"/>
 <contactref element="R5" pad="1"/>
-<wire x1="70.9168" y1="42.164" x2="74.2696" y2="42.164" width="0.2032" layer="1"/>
-<wire x1="70.7136" y1="42.3672" x2="70.9168" y2="42.164" width="0.2032" layer="1"/>
-<wire x1="74.2696" y1="42.164" x2="74.27971875" y2="42.09288125" width="0.2032" layer="1"/>
 </signal>
 <signal name="GND" class="2">
@@
 <wire x1="33.528" y1="68.7832" x2="33.34" y2="68.58" width="0.6096" layer="1"/>
 <wire x1="35.2552" y1="73.8632" x2="35.31" y2="73.92" width="0.6096" layer="1"/>
-<wire x1="28.2956" y1="25.146" x2="33.3248" y2="20.1168" width="0.6096" layer="1"/>
-<wire x1="33.3248" y1="20.1168" x2="33.327340625" y2="20.07108125" width="0.6096" layer="1"/>
+<wire x1="28.2956" y1="25.146" x2="33.610328125" y2="19.831271875" width="0.6096" layer="1"/>
+<wire x1="33.610328125" y1="19.831271875" x2="33.611821875" y2="19.80438125" width="0.6096" layer="1"/>
 <via x="65.9384" y="32.8168" extent="1-16" drill="0.6604"/>
 <via x="63.3984" y="50.3936" extent="1-16" drill="0.6604"/>
